Commit message: add tf and some modified urdf.

File: clc_test_gazebo/urdf/rrbot.xacro (robot description, xacro)
@@ -19,5 +19,5 @@
     <parent link="world"/>
     <child link="rect"/>
-    <origin xyz="0 0 0.00001" rpy="0 0 0"/>
+    <origin xyz="0 0 0.00001" rpy="0 ${PI} 0"/>
     <axis xyz="0 0 1"/>
   </joint>
@@ -127,4 +127,11 @@
     </inertial>
   </link>
+  <joint name="camera_link_frame_joint" type="fixed">
+    <axis xyz="0 1 0" />
+    <origin xyz="0 0 0" rpy="0 ${PI/2} 0"/>
+    <parent link="camera_link"/>
+    <child link="camera_frame"/>
+  </joint>
+  <link name="camera_frame"/>
   <transmission name="tran1">
     <type>transmission_interface/SimpleTransmission</type>

Commit message: 1. correct gazebo model 2. modifying perspective-to-euclidean transform

File: clc_test_gazebo/urdf/rrbot.xacro (robot description, xacro)
@@ -19,12 +19,12 @@
     <parent link="world"/>
     <child link="rect"/>
-    <origin xyz="0 0 0.00001" rpy="0 ${PI} 0"/>
+    <origin xyz="0.5 0.5 0.00000" rpy="0 0 -0.61546"/>
     <axis xyz="0 0 1"/>
   </joint>
   <link name="rect">
     <visual>
-      <origin xyz="0 0 0.01" rpy="0 0 0"/>
+      <origin xyz="0 0 0.01" rpy="0 0 0.61546"/>
       <geometry>
-	<box size="0.210 0.297 0.00002"/>
+        <box size="0.297 0.210 0.000001"/>
       </geometry>
       <material name="orange"/>
@@ -33,7 +33,6 @@
       <origin xyz="0 0 0" rpy="0 0 0"/>
       <geometry>
-	<box size="0.210 0.297 0.00002"/>
+        <box size="0.297 0.210 0.000001"/>
       </geometry>
-      <material name="red"/>
     </collision>
     <inertial>
@@ -42,5 +41,5 @@
       <inertia
 	  ixx="1.0" ixy="0.0" ixz="0.0"
-	  iyy="1.0" iyz="0.0"
+          iyy="1.0" iyz="0.0"
 	  izz="1.0"/>
     </inertial>
@@ -102,5 +101,5 @@
   <joint name="camera_joint" type="fixed">
     <axis xyz="0 1 0" />
-    <origin xyz="0 0 1" rpy="0 1.57079632 0"/>
+    <origin xyz="0 0 1" rpy="0 0 0"/>
     <parent link="link2"/>
     <child link="camera_link"/>
@@ -111,5 +110,5 @@
       <origin xyz="0 0 0" rpy="0 0 0"/>
       <geometry>
-	<box size="0.0474 0.157 0.036"/>
+        <box size="0.157 0.0474 0.036"/>
       </geometry>
     </collision>
@@ -117,5 +116,5 @@
       <origin xyz="0 0 0" rpy="0 0 0"/>
       <geometry>
-	<box size="0.0474 0.157 0.036"/>
+        <box size="0.157 0.0474 0.036"/>
       </geometry>
       <material name="red"/>
@@ -129,5 +128,5 @@
   <joint name="camera_link_frame_joint" type="fixed">
     <axis xyz="0 1 0" />
-    <origin xyz="0 0 0" rpy="0 ${PI/2} 0"/>
+    <origin xyz="0 0 0" rpy="${-PI} 0 ${PI}"/>
     <parent link="camera_link"/>
     <child link="camera_frame"/>

Commit message: complete motion control

File: clc_test_gazebo/urdf/rrbot.xacro (robot description, xacro)
@@ -19,5 +19,5 @@
     <parent link="world"/>
     <child link="rect"/>
-    <origin xyz="0.5 0.5 0.00000" rpy="0 0 -0.61546"/>
+    <origin xyz="0.15 0.45 0.00000" rpy="0 0 -0.61546"/>
     <axis xyz="0 0 1"/>
   </joint>
@@ -76,9 +76,9 @@
     <dynamics damping="0.7"/>
   </joint>
-  <link name="link2">
+  <link name="link3">
     <collision>
-      <origin xyz="0 0 0.5" rpy="0 0 0"/>
+      <origin xyz="0 0 0.05" rpy="0 0 0"/>
       <geometry>
-	<box size="0.001 0.001 1"/>
+	<box size="0.001 0.001 0.1"/>
       </geometry>
     </collision>
@@ -91,5 +91,5 @@
     </visual>
     <inertial>
-      <origin xyz="0 0 0.5" rpy="0 0 0"/>
+      <origin xyz="0 0 0.05" rpy="0 0 0"/>
       <mass value="1"/>
       <inertia
@@ -99,8 +99,26 @@
     </inertial>
   </link>
-  <joint name="camera_joint" type="fixed">
+  <link name="link2">
+    <inertial>
+      <origin xyz="0 0 0" rpy="0 0 0"/>
+      <mass value="1"/>
+      <inertia
+	  ixx="1.0" ixy="0.0" ixz="0.0"
+	  iyy="1.0" iyz="0.0"
+	  izz="1.0"/>
+    </inertial>
+  </link>
+  <joint name="joint3" type="prismatic">
+    <axis xyz="0 0 1"/>
+    <limit effort="1000" lower="-100" upper="100" velocity="10"/>
+    <dynamics damping="0" friction="0"/>
+    <origin xyz="0 0 0.001" rpy="0 0 0"/>
+    <parent link="link2"/>
+    <child link="link3"/>
+  </joint>
+    <joint name="camera_joint" type="fixed">
     <axis xyz="0 1 0" />
-    <origin xyz="0 0 1" rpy="0 0 0"/>
-    <parent link="link2"/>
+    <origin xyz="0 0 0.1" rpy="0 0 0"/>
+    <parent link="link3"/>
     <child link="camera_link"/>
   </joint>
@@ -153,3 +171,13 @@
     </actuator>
   </transmission>
+    <transmission name="joint3_tran3">
+    <type>transmission_interface/SimpleTransmission</type>
+    <joint name="joint3">
+      <hardwareInterface>EffortJointInterface</hardwareInterface>
+    </joint>
+    <actuator name="joint3_motor3">
+      <hardwareInterface>EffortJointInterface</hardwareInterface>
+      <mechanicalReduction>1</mechanicalReduction>
+    </actuator>
+  </transmission>
 </robot>
